Commit message: Add tcp-link

File: elfin_description/urdf/S20_with_base_gripper.urdf (robot description, URDF)
Before this commit: robot S20, 13 links, 12 joints
Links:
- added link tcp_link
Joints:
- added joint tcp_joint: type fixed, parent real_gripper, child tcp_link, origin xyz=0 0.45456 -0.02363 rpy=-0.5236 0 0

File: elfin_description/urdf/S20_with_gripper.urdf (robot description, URDF)
Before this commit: robot S20, 11 links, 10 joints
Links:
- added link tcp_link
Joints:
- added joint tcp_joint: type fixed, parent real_gripper, child tcp_link, origin xyz=0 0.45456 -0.02363 rpy=-0.5236 0 0

Commit message: Update base for S20_with_base_gripper

File: elfin_description/urdf/S20_with_base_gripper.urdf (robot description, URDF)
Before this commit: robot S20, 14 links, 13 joints
Links:
- link mobile_base_link1: geometry collision box size=0.01 0.01 0.01; visual box size=0.01 0.01 0.01
- link mobile_base_link2: geometry collision mesh filename=package://elfin_description/meshes/S20/chassis_sim.STL; visual mesh filename=package://elfin_description/meshes/S20/chassis_sim.STL
Joints:
- joint elfin_fixed_joint: origin xyz=0 0 1.18 rpy=0 0 0 -> xyz=0 0 0 rpy=-1.57 -3.14 0
- joint mobile_base_joint1: origin xyz=0 0 0 rpy=0 0 0 -> xyz=0 0.8 0 rpy=0 0 0
- joint mobile_base_joint2: axis 0 1 0 -> 0 0 1; origin xyz=0 0 0 rpy=0 0 0 -> xyz=0 -0.8 0.742 rpy=1.57 0 1.57

Commit message: Update after real robot experiment

File: elfin_description/urdf/S20_with_base_gripper.urdf (robot description, URDF)
Before this commit: robot S20, 14 links, 13 joints
Joints:
- joint elfin_fixed_joint: origin xyz=0 0 0 rpy=-1.57 -3.14 0 -> xyz=-0.05 0 0 rpy=-1.57 -3.14 0
- joint elfin_joint1: origin xyz=0 0 0.171 rpy=0 0 0 -> xyz=0 0 0.171 rpy=0 0 -1.57

Commit message: Update chassis model and tutorial

File: elfin_description/urdf/S20_with_base_gripper.urdf (robot description, URDF)
Before this commit: robot S20, 14 links, 13 joints
Joints:
- joint elfin_fixed_joint: origin xyz=-0.05 0 0 rpy=-1.57 -3.14 0 -> xyz=0 0 0 rpy=-1.57 -3.14 0
